File: _autosave-noob-sdr.kicad_pcb (KiCad board)
At the start: 6 copper layers, 130.3 x 97.2 mm, 468 parts, among them J1 GSG-USB-MICRO-B-SHIELDED, J2 CONN_1, J3 CONN_1, J4 CONN_1, J5 CONN_1, J6 CONN_1, J7 CONN_1, P1 CONN_1, P10 CONN_1, P11 CONN_1, P12 CONN_1, P13 CONN_1, P14 CONN_1, P15 CONN_1, P16 CONN_1, P17 CONN_1, P18 CONN_1, P19 CONN_1, P2 CONN_1, P20 CONN_1, P21 CONN_1, P22 CONN_1, P23 CONN_1, P24 CONN_1, P25 CONN_1, P26 CONN_1, P27 CONN_1, P28 CONN_1, P29 CONN_1, P3 CONN_1, P30 CONN_1, P31 CONN_1, P32 CONN_1, P33 CONN_1, P34 CONN_1, P35 CONN_1, P36 CONN_1, P37 CONN_1, P38 CONN_1, P39 CONN_1, P4 CONN_1, P40 CONN_1, P41 CONN_1, P42 CONN_1, P43 CONN_1, P44 CONN_1, P45 CONN_1, P46 CONN_1, P47 CONN_1, P48 CONN_1, P49 CONN_1, P5 CONN_1, P50 CONN_1, P51 CONN_1, P52 CONN_1, P53 CONN_1, P54 CONN_1, P55 CONN_1, P56 CONN_8x1, P57 CONN_1, P58 CLKIN, P59 CLKOUT, P6 ANTENNA, P60 CONN_1, P61 CONN_1, P62 CONN_1, P63 CONN_1, P64 CONN_1, P65 CONN_1, P66 CONN_1, P67 CONN_1, P68 CONN_1, P69 I2S, P7 CONN_1, P70 CONN_1, P71 GPIO, P72 LPC_JTAG, P73 CONN_1, P74 CONN_1, P75 CONN_11X2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

Commit message: Add files via upload
Noob-sdr v1.0
Parts:
- added C153: 10uF, gsg-modules:0805, F.Cu at (93.4, 32.7)
- added C188: 470nF, gsg-modules:0402, F.Cu at (134.8, 49.8)
- added FB1: FILTER, gsg-modules:0805, F.Cu at (94.2, 29.7)
- added Q7: MOSFET_P, gsg-modules:SOT23GDS, F.Cu at (97.1, 31.4)
- added R106: 10k, gsg-modules:0402, F.Cu at (97.1, 33.7)
- C147: value 4.7uF -> 100nF; footprint gsg-modules:0805 -> gsg-modules:0402
- C149, C165, C193, C194, C195, C199: footprint gsg-modules:0603 -> gsg-modules:0402; moved to B.Cu
- C150: value 10nF -> 100nF; footprint gsg-modules:0603 -> gsg-modules:0402; moved to B.Cu
- C152, C156, C157, C158, C160, C162, C178, C185, C198, FB4, FB5, R44, R47, R51, R62, R63, R92, R94, R97, R98, R99: moved to B.Cu
- C161: footprint gsg-modules:0402 -> Capacitors_SMD:C_1210
- C163, C167, C183, C184, C186: footprint gsg-modules:0805 -> gsg-modules:0402
- C164, C191, C192: footprint gsg-modules:0805 -> gsg-modules:0402; moved to B.Cu
- C166, C168, C169, C170, C171, C179, C180, C181, C182, C187, C196: footprint gsg-modules:0603 -> gsg-modules:0402
- C91: value 470nF -> 4.7uF
- P56: value CONN_8x1 -> BASEBAND; footprint gsg-modules:HEADER-1x8 -> gsg-modules:HEADER-2x8
- R100: moved to F.Cu
- moved D5 128.7 mm to (198.1, 78.8), turned to 90 degrees
- moved D4 128.0 mm to (198.1, 83.5), turned to 90 degrees
- moved R36 124.5 mm to (196.3, 80.5), turned to 0 degrees
- moved SW1 124.1 mm to (196.2, 71.3), turned to 90 degrees
- moved R35 124.0 mm to (196.3, 85.2), turned to 0 degrees
- moved R58 121.7 mm to (196.3, 75.5), turned to 0 degrees
- moved D6 117.2 mm to (186.8, 110.1), turned to 90 degrees
- moved R54 117.0 mm to (192.7, 70.8), turned to 180 degrees
- moved R37 113.8 mm to (185.0, 111.7), turned to 0 degrees
- moved D7 92.1 mm to (153.4, 26.6), turned to 180 degrees
- moved J4 91.0 mm to (282.0, 70.1)
- moved R38 90.3 mm to (155.2, 28.7), turned to 90 degrees
- moved C91 88.8 mm to (134.6, 43.7)
- moved R52 86.1 mm to (159.7, 46.0)
- moved J7 85.1 mm to (280.2, 62.4)
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Connections:
- C149 pad 2: GND -> XADCGND
- C91 pad 1: +1V8 -> VCC
- P56 pad 1: /baseband/RXBBQ- -> GND
- P56 pad 2: /baseband/RXBBQ+ -> GND
- P56 pad 3: /baseband/RXBBI- -> GND
- P56 pad 4: /baseband/RXBBI+ -> /baseband/RXBBQ-
- P56 pad 5: /baseband/TXBBI- -> /baseband/RXBBI-
- P56 pad 6: /baseband/TXBBI+ -> /baseband/RXBBQ+
- P56 pad 7: /baseband/TXBBQ+ -> /baseband/RXBBI+
- P56 pad 8: /baseband/TXBBQ- -> GND
- P71 pad 17: FPGA_TCK -> Net-(P71-Pad17)
- P71 pad 20: MGTAVTT -> Net-(P71-Pad20)
- P71 pad 21: Net-(P71-Pad21) -> FPGA_TCK
- U21 pad 37: Net-(U21-Pad37) -> !VAA_ENABLE
- U22 pad A14: HOST_DATA7 -> HOST_CAPTURE
- U22 pad A15: HOST_DATA6 -> HOST_DATA0
- U22 pad A16: HOST_DATA3 -> HOST_DECIM_SEL2
- U22 pad A18: Net-(U22-PadA18) -> HOST_DATA5
- U22 pad B1: MGTAVTT -> GND
- U22 pad B15: HOST_DATA4 -> HOST_DATA1
- U22 pad B16: HOST_DATA0 -> HOST_DATA7
- U22 pad B18: Net-(U22-PadB18) -> HOST_DATA6
- U22 pad C15: HOST_DATA5 -> HOST_DATA3
- U22 pad C16: HOST_DATA1 -> HOST_DATA4
- U22 pad C5: MGTAVTT -> GND
- U22 pad E2: MGTAVTT -> GND
- U22 pad G7: MGTAVTT -> GND
- U22 pad K17: /fpga/SRAM-A2 -> /fpga/SRAM-A9
- U22 pad M18: /fpga/SRAM-A0 -> /fpga/SRAM-A11
- U22 pad M19: /fpga/SRAM-A1 -> /fpga/SRAM-A10
- U22 pad N17: /fpga/SRAM-A3 -> /fpga/SRAM-DQ7
- U22 pad N19: /fpga/SRAM-CE -> /fpga/SRAM-A13
- U22 pad P17: /fpga/SRAM-A4 -> /fpga/SRAM-CE
- U22 pad P18: /fpga/SRAM-A5 -> /fpga/SRAM-A14
- U22 pad R18: /fpga/SRAM-A6 -> /fpga/SRAM-A12
- U22 pad R19: /fpga/SRAM-WE -> /fpga/SRAM-A16
- U22 pad T17: /fpga/SRAM-A11 -> /fpga/SRAM-A15
- U22 pad T18: /fpga/SRAM-A12 -> /fpga/SRAM-DQ3
- U22 pad U14: /fpga/SRAM-DQ7 -> /fpga/SRAM-WE
- U22 pad U15: /fpga/SRAM-DQ3 -> /fpga/SRAM-A7
- U22 pad U16: /fpga/SRAM-DQ4 -> /fpga/SRAM-DQ0
- U22 pad U17: /fpga/SRAM-A13 -> /fpga/SRAM-A17
- U22 pad U18: /fpga/SRAM-A14 -> /fpga/SRAM-DQ2
- U22 pad U19: /fpga/SRAM-A8 -> /fpga/SRAM-DQ6
- U22 pad U5: HOST_CAPTURE -> DA3
- U22 pad V13: /fpga/SRAM-DQ5 -> /fpga/SRAM-A0
- U22 pad V14: /fpga/SRAM-DQ6 -> /fpga/SRAM-A8
- U22 pad V15: /fpga/SRAM-A18 -> /fpga/SRAM-A1
- U22 pad V16: /fpga/SRAM-A15 -> /fpga/SRAM-A5
- U22 pad V17: Net-(U22-PadV17) -> /fpga/SRAM-A2
- U22 pad V19: /fpga/SRAM-A9 -> /fpga/SRAM-A18
- U22 pad V5: HOST_DECIM_SEL2 -> DA1
- U22 pad W13: /fpga/SRAM-DQ1 -> /fpga/SRAM-A6
- U22 pad W14: /fpga/SRAM-DQ2 -> /fpga/SRAM-A3
- U22 pad W15: /fpga/SRAM-DQ0 -> /fpga/SRAM-A4
- U22 pad W16: /fpga/SRAM-A16 -> /fpga/SRAM-DQ5
- U22 pad W17: /fpga/SRAM-A17 -> /fpga/SRAM-DQ4
- U22 pad W18: /fpga/SRAM-A10 -> Net-(U22-PadW18)
- U22 pad W19: /fpga/SRAM-A7 -> /fpga/SRAM-DQ1
- U22 pad W5: DA3 -> DA0
- U22 pad W6: DA0 -> Net-(U22-PadW6)
- U22 pad W7: DA1 -> Net-(U22-PadW7)
Routing:
- net VCC: track 146.3 -> 358.9 mm, vias 36 -> 87
- net +1V8: track 15.7 -> 175.0 mm, vias 2 -> 9
- net RX_MIX_BP: track 9.16 -> 164.0 mm, vias 1 -> 2
- net GND: track 330.1 -> 484.7 mm, vias 198 -> 287
- net SSP1_MOSI: track 34.1 -> 162.3 mm, vias 2 -> 3
- net SSP1_SCK: track 4.85 -> 119.4 mm, vias 1 -> 3
- net !VAA_ENABLE: track 0.00 -> 106.5 mm, vias 0 -> 2
- net CS_AD: track 4.28 -> 99.8 mm, vias 0 -> 2
- net /mcu/usb/SGPIO13: track 0.00 -> 81.1 mm, vias 0 -> 2
- net /mcu/usb/SGPIO9: track 0.00 -> 80.4 mm, vias 0 -> 2
- net FPGA_TMS: track 2.48 -> 81.4 mm, vias 1 -> 2
- net /mcu/usb/SGPIO14: track 0.00 -> 77.2 mm, vias 0 -> 3
- net FPGA_TCK: track 0.00 -> 77.0 mm, vias 0 -> 4
- net TXENABLE: track 4.54 -> 79.5 mm, vias 1 -> 2
- net /mcu/usb/SGPIO0: track 0.00 -> 74.7 mm, vias 0 -> 2
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- added copper zone on VAUX, net +1V0
- removed copper zone on V1.0, net +1V0
- removed copper zone on V1.8, net +1V8
Other:
- board size 130.3 x 97.2 mm -> 130.3 x 100 mm
- net class Default: clearance 0.0762 -> 0.0508
- rule trace_clearance: 0.0762 -> 0.0508
- rule trace_min: 0.127 -> 0.0762
