File: baseband.sch (KiCad schematic (older format))
At the start: 115 parts, among them P25 CONN_1, P26 CONN_1, P27 CONN_1, P28 CONN_1, P29 CONN_1, P30 CONN_1, P31 CONN_1, P32 CONN_1, P33 CONN_1, P34 CONN_1, P35 CONN_1, P36 CONN_1, P37 CONN_1, P38 CONN_1, P39 CONN_1, P40 CONN_1, P41 CONN_1, P42 CONN_1, P43 CONN_1, P44 CONN_1, P45 CONN_1, P46 CONN_1, P47 CONN_1, P48 CONN_1, P49 CONN_1, P50 CONN_1, P51 CONN_1, P52 CONN_1, P53 CONN_1, P54 CONN_1, P55 CONN_1, P56 CONN_8x1, P57 CONN_1, P58 CLKIN, P59 CLKOUT, P60 CONN_1, T3 RX_BALUN, T4 TX_BALUN, U16 MAX5864, U17 MAX2837, U18 SI5351C, X1 GSG-XTAL4PIN

Commit message: Add files via upload
Noob-sdr v1.0
Parts:
- removed P56: CONN_8x1, gsg-modules:HEADER-1x8, symbol CONN_8x1
- added C147: 100nF, gsg-modules:0402, symbol C
- added C153: 10uF, gsg-modules:0805, symbol C
- added FB1: FILTER, gsg-modules:0805, symbol FILTER
- added P56: BASEBAND, gsg-modules:HEADER-2x8, symbol CONN_8X2
- added Q7: MOSFET_P, gsg-modules:SOT23GDS, symbol MOSFET_P
- added R106: 10k, gsg-modules:0402, symbol R
Connections:
- net GND: now also C147.2, C153.2, P56.1, P56.14, P56.15, P56.16, P56.2, P56.3, P56.8, P56.9
- net RXBBI+: now also P56.7
- net RXBBI-: now also P56.5
- net RXBBQ+: now also P56.6
- net RXBBQ-: now also P56.4
- net TXBBI+: now also P56.12
- net TXBBI-: now also P56.10
- net TXBBQ+: now also P56.11
- net TXBBQ-: now also P56.13
- net VAA: now also C153.1, FB1.2
- net VCC: now also C147.1, Q7.S, R106.1
- new net: FB1.1, Q7.D
- new net !VAA_ENABLE: Q7.G, R106.2
Changed lines of the file:
@@
 	5000 7225 5000 7275
 Wire Wire Line
-	6725 7675 4775 7675
-Wire Wire Line
-	6725 7775 4775 7775
-Wire Wire Line
-	6725 7875 4775 7875
+	4775 7675 6725 7675
+Wire Wire Line
+	4775 7775 6725 7775
+Wire Wire Line
+	4775 7875 6725 7875
 Wire Wire Line
 	5350 7575 5350 7675
@@
 $EndComp
 Wire Wire Line
-	9050 9175 8125 9175
+	8125 9175 9050 9175
 Wire Wire Line
 	8850 9275 8850 9175
@@
 Wire Wire Line
 	12175 7250 12175 7425
-Text Label 13800 7300 2    40   ~ 0
+Text Label 13435 8180 0    40   ~ 0
 RXBBI-
-Text Label 13800 7400 2    40   ~ 0
+Text Label 13435 8280 0    40   ~ 0
 RXBBI+
-Text Label 13800 7700 2    40   ~ 0
+Text Label 13435 8480 0    40   ~ 0
 TXBBQ+
-Text Label 13800 7800 2    40   ~ 0
+Text Label 13435 8580 0    40   ~ 0
 TXBBQ-
-Text Label 13800 7100 2    40   ~ 0
+Text Label 14965 8080 2    40   ~ 0
 RXBBQ-
-Text Label 13800 7200 2    40   ~ 0
+Text Label 14965 8180 2    40   ~ 0
 RXBBQ+
-Text Label 13800 7600 2    40   ~ 0
+Text Label 14965 8480 2    40   ~ 0
 TXBBI+
-Text Label 13800 7500 2    40   ~ 0
+Text Label 14965 8380 2    40   ~ 0
 TXBBI-
 $Comp
@@
 	8425 4625 8750 4625
 Connection ~ 8550 4625
-Wire Wire Line
-	13800 7100 13900 7100
-Wire Wire Line
-	13900 7200 13800 7200
-Wire Wire Line
-	13800 7300 13900 7300
-Wire Wire Line
-	13900 7400 13800 7400
-$Comp
-L CONN_8x1 P56
-U 1 1 587E710E
-P 14200 7450
-F 0 "P56" H 14190 7100 60  0000 C CNN
-F 1 "CONN_8x1" V 14210 7480 60  0000 C CNN
-F 2 "gsg-modules:HEADER-1x8" H 14430 7190 60  0001 C CNN
-F 3 "" H 14430 7190 60  0001 C CNN
-	1    14200 7450
-	1    0    0    -1
-$EndComp
-Wire Wire Line
-	13800 7500 13900 7500
-Wire Wire Line
-	13900 7600 13800 7600
-Wire Wire Line
-	13800 7700 13900 7700
-Wire Wire Line
-	13800 7800 13900 7800
+Text GLabel 6050 2375 2    50   Input ~ 0
+!VAA_ENABLE
+$Comp
+L MOSFET_P Q7
+U 1 1 589F1F60
+P 5225 2375
+F 0 "Q7" H 5225 2565 60  0000 R CNN
+F 1 "MOSFET_P" H 5225 2195 60  0000 R CNN
+F 2 "gsg-modules:SOT23GDS" H 5225 2375 60  0001 C CNN
+F 3 "" H 5225 2375 60  0000 C CNN
+	1    5225 2375
+	-1   0    0    1
+$EndComp
+$Comp
+L R R106
+U 1 1 589F2A3F
+P 5475 1950
+F 0 "R106" V 5510 1780 50  0000 C CNN
+F 1 "10k" V 5475 1950 40  0000 C CNN
+F 2 "gsg-modules:0402" V 5405 1950 50  0001 C CNN
+F 3 "" H 5475 1950 50  0000 C CNN
+	1    5475 1950
+	0    -1   -1   0
+$EndComp
+$Comp
+L C C147
+U 1 1 589F4B8C
+P 4575 2100
+F 0 "C147" H 4600 2200 50  0000 L CNN
+F 1 "100nF" H 4600 2000 40  0000 L CNN
+F 2 "gsg-modules:0402" H 4613 1950 50  0001 C CNN
+F 3 "" H 4575 2100 50  0000 C CNN
+	1    4575 2100
+	1    0    0    -1
+$EndComp
+$Comp
+L FILTER FB1
+U 1 1 589F59BB
+P 5125 3050
+F 0 "FB1" H 5125 3200 50  0000 C CNN
+F 1 "FILTER" H 5125 2950 50  0000 C CNN
+F 2 "gsg-modules:0805" H 5125 3050 50  0001 C CNN
+F 3 "" H 5125 3050 50  0000 C CNN
+	1    5125 3050
+	0    1    1    0
+$EndComp
+$Comp
+L C C153
+U 1 1 589F5B81
+P 5125 3700
+F 0 "C153" H 5150 3800 50  0000 L CNN
+F 1 "10uF" H 5150 3600 40  0000 L CNN
+F 2 "gsg-modules:0805" H 5163 3550 50  0001 C CNN
+F 3 "" H 5125 3700 50  0000 C CNN
+	1    5125 3700
+	1    0    0    -1
+$EndComp
+$Comp
+L VAA #PWR0173
+U 1 1 589F667E
+P 5700 3475
+F 0 "#PWR0173" H 5700 3325 50  0001 C CNN
+F 1 "VAA" H 5700 3625 50  0000 C CNN
+F 2 "" H 5700 3475 50  0000 C CNN
+F 3 "" H 5700 3475 50  0000 C CNN
+	1    5700 3475
+	0    1    1    0
+$EndComp
+Wire Wire Line
+	5425 2375 6050 2375
+Wire Wire Line
+	5125 1650 5125 2175
+Wire Wire Line
+	5125 1950 5325 1950
+Wire Wire Line
+	5625 1950 5725 1950
+Wire Wire Line
+	5725 1950 5725 2375
+Connection ~ 5725 2375
+$Comp
+L VCC #PWR0174
+U 1 1 589FBEF1
+P 5125 1650
+F 0 "#PWR0174" H 5125 1500 50  0001 C CNN
+F 1 "VCC" H 5125 1800 50  0000 C CNN
+F 2 "" H 5125 1650 50  0000 C CNN
+F 3 "" H 5125 1650 50  0000 C CNN
+	1    5125 1650
+	1    0    0    -1
+$EndComp
+$Comp
+L GND #PWR0175
+U 1 1 589FDA2C
+P 4575 2425
+F 0 "#PWR0175" H 4575 2175 50  0001 C CNN
+F 1 "GND" H 4575 2275 50  0000 C CNN
+F 2 "" H 4575 2425 50  0000 C CNN
+F 3 "" H 4575 2425 50  0000 C CNN
+	1    4575 2425
+	1    0    0    -1
+$EndComp
+Wire Wire Line
+	4575 2425 4575 2250
+Connection ~ 5125 1950
+Wire Wire Line
+	4575 1950 4575 1800
+Wire Wire Line
+	4575 1800 5125 1800
+Connection ~ 5125 1800
+Wire Wire Line
+	5125 2575 5125 2700
+$Comp
+L GND #PWR0176
+U 1 1 58A01B1B
+P 5125 4025
+F 0 "#PWR0176" H 5125 3775 50  0001 C CNN
+F 1 "GND" H 5125 3875 50  0000 C CNN
+F 2 "" H 5125 4025 50  0000 C CNN
+F 3 "" H 5125 4025 50  0000 C CNN
+	1    5125 4025
+	1    0    0    -1
+$EndComp
+Wire Wire Line
+	5125 3400 5125 3550
+Wire Wire Line
+	5125 4025 5125 3850
+Wire Wire Line
+	5700 3475 5125 3475
+Connection ~ 5125 3475
+$Comp
+L CONN_8X2 P56
+U 1 1 58A2AEAA
+P 14200 8330
+F 0 "P56" H 14200 8780 60  0000 C CNN
+F 1 "BASEBAND" V 14200 8330 50  0000 C CNN
+F 2 "gsg-modules:HEADER-2x8" H 14200 8330 60  0001 C CNN
+F 3 "" H 14200 8330 60  0000 C CNN
+	1    14200 8330
+	1    0    0    -1
+$EndComp
+Wire Wire Line
+	13720 8080 13800 8080
+Wire Wire Line
+	13435 8180 13800 8180
+Wire Wire Line
+	13800 7980 13720 7980
+Wire Wire Line
+	13800 8280 13435 8280
+Wire Wire Line
+	13720 8380 13800 8380
+Wire Wire Line
+	13800 8480 13435 8480
+Wire Wire Line
+	13800 8580 13435 8580
+Wire Wire Line
+	13720 8680 13800 8680
+Wire Wire Line
+	14600 7980 14680 7980
+Wire Wire Line
+	14600 8080 14965 8080
+Wire Wire Line
+	14600 8180 14965 8180
+Wire Wire Line
+	14600 8280 14680 8280
+Wire Wire Line
+	14600 8380 14965 8380
+Wire Wire Line
+	14600 8480 14965 8480
+Wire Wire Line
+	14680 8580 14600 8580
+Wire Wire Line
+	14680 8680 14600 8680
+$Comp
+L GND #PWR0177
+U 1 1 58A42571
+P 13720 8855
+F 0 "#PWR0177" H 13720 8605 50  0001 C CNN
+F 1 "GND" H 13720 8705 50  0000 C CNN
+F 2 "" H 13720 8855 50  0000 C CNN
+F 3 "" H 13720 8855 50  0000 C CNN
+	1    13720 8855
+	1    0    0    -1
+$EndComp
+$Comp
+L GND #PWR0178
+U 1 1 58A42AAF
+P 14680 8840
+F 0 "#PWR0178" H 14680 8590 50  0001 C CNN
+F 1 "GND" H 14680 8690 50  0000 C CNN
+F 2 "" H 14680 8840 50  0000 C CNN
+F 3 "" H 14680 8840 50  0000 C CNN
+	1    14680 8840
+	1    0    0    -1
+$EndComp
+Wire Wire Line
+	13720 7980 13720 8855
+Connection ~ 13720 8080
+Connection ~ 13720 8380
+Connection ~ 13720 8680
+Wire Wire Line
+	14680 7980 14680 8840
+Connection ~ 14680 8280
+Connection ~ 14680 8580
+Connection ~ 14680 8680
 $EndSCHEMATC
