File: fpga.sch (KiCad schematic (older format))
At the start: 59 parts, among them U22 XC7A15T-1CPG236C, U23 IS61WV5128BLL-10BLI

Commit message: Add files via upload
Noob-sdr v1.0
Parts:
- removed C147: 4.7uF, gsg-modules:0805, symbol C
- added C188: 470nF, gsg-modules:0402, symbol C
- C149, C165, C166, C168, C169, C170, C171, C179, C180, C181, C182, C187, C193, C194, C195, C196, C199: footprint gsg-modules:0603 -> gsg-modules:0402
- C150: value 10nF -> 100nF; footprint gsg-modules:0603 -> gsg-modules:0402
- C161: footprint gsg-modules:0402 -> Capacitors_SMD:C_1210
- C163, C164, C167, C183, C184, C186, C191, C192: footprint gsg-modules:0805 -> gsg-modules:0402
- C91: value 470nF -> 4.7uF
Connections:
- net MGTAVTT is gone; now on net GND: U22.B1 (MGTAVTT), U22.C5 (MGTAVTT), U22.E2 (MGTAVTT), U22.G7 (MGTAVTT)
- net +1V8: now also C188.1; no longer C91.1
- net DA0: now also U22.W5 (IO_L12P_T1_MRCC_34); no longer U22.W6 (IO_L13N_T2_MRCC_34)
- net DA1: now also U22.V5 (IO_L16N_T2_34); no longer U22.W7 (IO_L13P_T2_MRCC_34)
- net DA3: now also U22.U5 (IO_L16P_T2_34); no longer U22.W5 (IO_L12P_T1_MRCC_34)
- net GND: now also C188.2; no longer C149.2
- net HOST_CAPTURE: now also U22.A14 (IO_L6P_T0_16); no longer U22.U5 (IO_L16P_T2_34)
- net HOST_DATA0: now also U22.A15 (IO_L6N_T0_VREF_16); no longer U22.B16 (IO_L13N_T2_MRCC_16)
- net HOST_DATA1: now also U22.B15 (IO_L11N_T1_SRCC_16); no longer U22.C16 (IO_L13P_T2_MRCC_16)
- net HOST_DATA3: now also U22.C15 (IO_L11P_T1_SRCC_16); no longer U22.A16 (IO_L12P_T1_MRCC_16)
- net HOST_DATA4: now also U22.C16 (IO_L13P_T2_MRCC_16); no longer U22.B15 (IO_L11N_T1_SRCC_16)
- net HOST_DATA5: now also U22.A18 (IO_L19N_T3_VREF_16); no longer U22.C15 (IO_L11P_T1_SRCC_16)
- net HOST_DATA6: now also U22.B18 (IO_L19P_T3_16); no longer U22.A15 (IO_L6N_T0_VREF_16)
- net HOST_DATA7: now also U22.B16 (IO_L13N_T2_MRCC_16); no longer U22.A14 (IO_L6P_T0_16)
- net HOST_DECIM_SEL2: now also U22.A16 (IO_L12P_T1_MRCC_16); no longer U22.V5 (IO_L16N_T2_34)
- net SRAM-A0: now also U22.V13 (IO_L24P_T3_A01_D17_14); no longer U22.M18 (IO_L11P_T1_SRCC_14)
- net SRAM-A1: now also U22.V15 (IO_L21P_T3_DQS_14); no longer U22.M19 (IO_L11N_T1_SRCC_14)
- net SRAM-A10: now also U22.M19 (IO_L11N_T1_SRCC_14); no longer U22.W18 (IO_L16P_T2_CSI_B_14)
- net SRAM-A11: now also U22.M18 (IO_L11P_T1_SRCC_14); no longer U22.T17 (IO_L17P_T2_A14_D30_14)
- net SRAM-A12: now also U22.R18 (IO_L14N_T2_SRCC_14); no longer U22.T18 (IO_L17N_T2_A13_D29_14)
- net SRAM-A13: now also U22.N19 (IO_L9N_T1_DQS_D13_14); no longer U22.U17 (IO_L18P_T2_A12_D28_14)
- net SRAM-A14: now also U22.P18 (IO_L14P_T2_SRCC_14); no longer U22.U18 (IO_L18N_T2_A11_D27_14)
- net SRAM-A15: now also U22.T17 (IO_L17P_T2_A14_D30_14); no longer U22.V16 (IO_L19P_T3_A10_D26_14)
- net SRAM-A16: now also U22.R19 (IO_L10N_T1_D15_14); no longer U22.W16 (IO_L20P_T3_A08_D24_14)
- net SRAM-A17: now also U22.U17 (IO_L18P_T2_A12_D28_14); no longer U22.W17 (IO_L20N_T3_A07_D23_14)
- net SRAM-A18: now also U22.V19 (IO_L15N_T2_DQS_DOUT_CSO_B_14); no longer U22.V15 (IO_L21P_T3_DQS_14)
- net SRAM-A2: now also U22.V17 (IO_L19N_T3_A09_D25_VREF_14); no longer U22.K17 (IO_L12N_T1_MRCC_14)
- net SRAM-A3: now also U22.W14 (IO_L22N_T3_A04_D20_14); no longer U22.N17 (IO_L13P_T2_MRCC_14)
- net SRAM-A4: now also U22.W15 (IO_L21N_T3_DQS_A06_D22_14); no longer U22.P17 (IO_L13N_T2_MRCC_14)
- net SRAM-A5: now also U22.V16 (IO_L19P_T3_A10_D26_14); no longer U22.P18 (IO_L14P_T2_SRCC_14)
- net SRAM-A6: now also U22.W13 (IO_L22P_T3_A05_D21_14); no longer U22.R18 (IO_L14N_T2_SRCC_14)
- net SRAM-A7: now also U22.U15 (IO_L23P_T3_A03_D19_14); no longer U22.W19 (IO_L16N_T2_A15_D31_14)
- net SRAM-A8: now also U22.V14 (IO_L24N_T3_A00_D16_14); no longer U22.U19 (IO_L15P_T2_DQS_RDWR_B_14)
- net SRAM-A9: now also U22.K17 (IO_L12N_T1_MRCC_14); no longer U22.V19 (IO_L15N_T2_DQS_DOUT_CSO_B_14)
- net SRAM-CE: now also U22.P17 (IO_L13N_T2_MRCC_14); no longer U22.N19 (IO_L9N_T1_DQS_D13_14)
- net SRAM-DQ0: now also U22.U16 (IO_L23N_T3_A02_D18_14); no longer U22.W15 (IO_L21N_T3_DQS_A06_D22_14)
- net SRAM-DQ1: now also U22.W19 (IO_L16N_T2_A15_D31_14); no longer U22.W13 (IO_L22P_T3_A05_D21_14)
- net SRAM-DQ2: now also U22.U18 (IO_L18N_T2_A11_D27_14); no longer U22.W14 (IO_L22N_T3_A04_D20_14)
- net SRAM-DQ3: now also U22.T18 (IO_L17N_T2_A13_D29_14); no longer U22.U15 (IO_L23P_T3_A03_D19_14)
- net SRAM-DQ4: now also U22.W17 (IO_L20N_T3_A07_D23_14); no longer U22.U16 (IO_L23N_T3_A02_D18_14)
- net SRAM-DQ5: now also U22.W16 (IO_L20P_T3_A08_D24_14); no longer U22.V13 (IO_L24P_T3_A01_D17_14)
- net SRAM-DQ6: now also U22.U19 (IO_L15P_T2_DQS_RDWR_B_14); no longer U22.V14 (IO_L24N_T3_A00_D16_14)
- net SRAM-DQ7: now also U22.N17 (IO_L13P_T2_MRCC_14); no longer U22.U14 (IO_25_14)
- net SRAM-WE: now also U22.U14 (IO_25_14); no longer U22.R19 (IO_L10N_T1_D15_14)
- net VCC: now also C91.1
- net XADCGND: now also C149.2
Other:
- moved on the sheet: C148, C155, C156, C157, C158, C159, C160, C161, C162, C163, C164, C165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
