File: frontend.sch (KiCad schematic (older format))
At the start: 139 parts, among them J2 CONN_1, J3 CONN_1, J4 CONN_1, J5 CONN_1, J6 CONN_1, J7 CONN_1, P1 CONN_1, P10 CONN_1, P11 CONN_1, P12 CONN_1, P13 CONN_1, P14 CONN_1, P15 CONN_1, P16 CONN_1, P17 CONN_1, P18 CONN_1, P19 CONN_1, P2 CONN_1, P20 CONN_1, P21 CONN_1, P22 CONN_1, P23 CONN_1, P24 CONN_1, P3 CONN_1, P4 CONN_1, P5 CONN_1, P6 ANTENNA, P7 CONN_1, P8 CONN_1, P9 CONN_1, Q1 MOSFET_P, Q2 MOSFET_P, Q3 MOSFET_P, T1 MIX_IN_BALUN, T2 MIX_OUT_BALUN, U1 SKY13350, U10 SKY13350, U11 SKY13350, U12 MGA-81563, U13 SKY13317, U14 SKY13317, U15 MGA-81563, U2 RFFC5072, U3 SKY13350, U4 SKY13350, U5 SKY13317, U6 RX_LOWPASS_FILTER, U7 SKY13350, U8 SKY13350, U9 RX_HIGHPASS_FILTER

Commit message: Add files via upload
Noob-sdr v1.0
Parts:
- C1, C11, C25, C3, C40, C48, C57: Description (none) -> CAP CER 33PF 50V 5% NP0 0402; Manufacturer (none) -> Murata; Part Number (none) -> GRM1555C1H330JA01D
- C14, C21: Description (none) -> CAP CER 0.1UF 10V 10% X5R 0402; Manufacturer (none) -> Murata; Part Number (none) -> GRM155R61A104KA01D
- C2, C39, C43, C6: Description (none) -> CAP CER 22PF 50V 5% NP0 0402; Manufacturer (none) -> Murata; Part Number (none) -> GRM1555C1H220JA01D
- C58: Description (none) -> CAP CER 10000PF 16V 10% X7R 0402; Manufacturer (none) -> Murata; Part Number (none) -> GRM155R71C103KA01D
- D1: Description (none) -> TVS DIODE ESD .05PF 15KV 0402; Manufacturer (none) -> Murata; Part Number (none) -> LXES15AAA1-100
- Q3: Description (none) -> MOSFET P-CH 50V 130MA SOT-23; Manufacturer (none) -> Fairchild; Part Number (none) -> BSS84
- T1, T2: Description (none) -> Ultra Low Profile 0805 Balun 50 to 100 ohm Balanced; Manufacturer (none) -> Anaren; Part Number (none) -> B0310J50100AHF
- U1, U10, U11, U3, U4, U7, U8: Description (none) -> 0.01-6.0 GHz GaAs SPDT Switch; Manufacturer (none) -> Skyworks; Part Number (none) -> SKY13350-385LF
- U13, U5: Description (none) -> 20 MHz-6.0 GHz pHEMT GaAs SP3T Switch; Manufacturer (none) -> Skyworks; Part Number (none) -> SKY13317-373LF
- U6: Description (none) -> FILTER LOW PASS 1880MHZ 0603 SMD; Manufacturer (none) -> AVX; Part Number (none) -> LP0603A1880ANTR
- U9: Description (none) -> FILTER HIGHPASS WLAN&BLUETOOTH; Manufacturer (none) -> TDK; Part Number (none) -> DEA162400HT-8004B1
Changed lines of the file:
@@
 F 2 "gsg-modules:SKY13350-385LF" H 1575 1450 60  0001 C CNN
 F 3 "" H 1575 1450 60  0000 C CNN
+F 4 "Skyworks" H 1575 1450 60  0001 C CNN "Manufacturer"
+F 5 "SKY13350-385LF" H 1575 1450 60  0001 C CNN "Part Number"
+F 6 "0.01-6.0 GHz GaAs SPDT Switch" H 1575 1450 60  0001 C CNN "Description"
 	1    1575 1450
 	0    -1   -1   0
@@
 F 2 "gsg-modules:SKY13350-385LF" H 2550 3475 60  0001 C CNN
 F 3 "" H 2550 3475 60  0000 C CNN
+F 4 "Skyworks" H 2550 3475 60  0001 C CNN "Manufacturer"
+F 5 "SKY13350-385LF" H 2550 3475 60  0001 C CNN "Part Number"
+F 6 "0.01-6.0 GHz GaAs SPDT Switch" H 2550 3475 60  0001 C CNN "Description"
 	1    2550 3475
 	0    1    1    0
@@
 F 2 "gsg-modules:SKY13350-385LF" H 9875 4250 60  0001 C CNN
 F 3 "" H 9875 4250 60  0000 C CNN
+F 4 "Skyworks" H 9875 4250 60  0001 C CNN "Manufacturer"
+F 5 "SKY13350-385LF" H 9875 4250 60  0001 C CNN "Part Number"
+F 6 "0.01-6.0 GHz GaAs SPDT Switch" H 9875 4250 60  0001 C CNN "Description"
 	1    9875 4250
 	0    -1   -1   0
@@
 F 2 "gsg-modules:SKY13350-385LF" H 9200 3350 60  0001 C CNN
 F 3 "" H 9200 3350 60  0000 C CNN
+F 4 "Skyworks" H 9200 3350 60  0001 C CNN "Manufacturer"
+F 5 "SKY13350-385LF" H 9200 3350 60  0001 C CNN "Part Number"
+F 6 "0.01-6.0 GHz GaAs SPDT Switch" H 9200 3350 60  0001 C CNN "Description"
 	1    9200 3350
 	0    1    1    0
@@
 F 2 "gsg-modules:0402" H 1138 725 50  0001 C CNN
 F 3 "" H 1100 875 50  0000 C CNN
+F 4 "Murata" H 1100 875 60  0001 C CNN "Manufacturer"
+F 5 "GRM1555C1H220JA01D" H 1100 875 60  0001 C CNN "Part Number"
+F 6 "CAP CER 22PF 50V 5% NP0 0402" H 1100 875 60  0001 C CNN "Description"
 	1    1100 875
 	0    1    1    0
@@
 F 2 "gsg-modules:0402" H 1913 625 50  0001 C CNN
 F 3 "" H 1875 775 50  0000 C CNN
+F 4 "Murata" H 1875 775 60  0001 C CNN "Manufacturer"
+F 5 "GRM1555C1H330JA01D" H 1875 775 60  0001 C CNN "Part Number"
+F 6 "CAP CER 33PF 50V 5% NP0 0402" H 1875 775 60  0001 C CNN "Description"
 	1    1875 775
 	0    1    1    0
@@
 F 2 "gsg-modules:0402" H 1038 1850 50  0001 C CNN
 F 3 "" H 1000 2000 50  0000 C CNN
+F 4 "Murata" H 1000 2000 60  0001 C CNN "Manufacturer"
+F 5 "GRM1555C1H330JA01D" H 1000 2000 60  0001 C CNN "Part Number"
+F 6 "CAP CER 33PF 50V 5% NP0 0402" H 1000 2000 60  0001 C CNN "Description"
 	1    1000 2000
 	0    -1   -1   0
@@
 F 2 "noob:GSG-B0310J50100AHF" H 3425 4050 60  0001 C CNN
 F 3 "" H 3425 4050 60  0000 C CNN
+F 4 "Anaren" H 3425 4050 60  0001 C CNN "Manufacturer"
+F 5 "B0310J50100AHF" H 3425 4050 60  0001 C CNN "Part Number"
+F 6 "Ultra Low Profile 0805 Balun 50 to 100 ohm Balanced" H 3425 4050 60  0001 C CNN "Description"
 	1    3425 4050
 	-1   0    0    1
@@
 F 2 "gsg-modules:0402" H 3163 3425 50  0001 C CNN
 F 3 "" H 3125 3575 50  0000 C CNN
+F 4 "Murata" H 3125 3575 60  0001 C CNN "Manufacturer"
+F 5 "GRM155R61A104KA01D" H 3125 3575 60  0001 C CNN "Part Number"
+F 6 "CAP CER 0.1UF 10V 10% X5R 0402" H 3125 3575 60  0001 C CNN "Description"
 	1    3125 3575
 	1    0    0    -1
@@
 F 2 "gsg-modules:0402" H 2838 4000 50  0001 C CNN
 F 3 "" H 2800 4150 50  0000 C CNN
+F 4 "Murata" H 2800 4150 60  0001 C CNN "Manufacturer"
+F 5 "GRM155R61A104KA01D" H 2800 4150 60  0001 C CNN "Part Number"
+F 6 "CAP CER 0.1UF 10V 10% X5R 0402" H 2800 4150 60  0001 C CNN "Description"
 	1    2800 4150
 	0    1    1    0
@@
 F 2 "gsg-modules:0402" H 2588 4225 50  0001 C CNN
 F 3 "" H 2550 4375 50  0000 C CNN
+F 4 "Murata" H 2550 4375 60  0001 C CNN "Manufacturer"
+F 5 "GRM1555C1H330JA01D" H 2550 4375 60  0001 C CNN "Part Number"
+F 6 "CAP CER 33PF 50V 5% NP0 0402" H 2550 4375 60  0001 C CNN "Description"
 	1    2550 4375
 	-1   0    0    1
@@
 F 2 "gsg-modules:0402" H 1613 2425 50  0001 C CNN
 F 3 "" H 1575 2575 50  0000 C CNN
+F 4 "Murata" H 1575 2575 60  0001 C CNN "Manufacturer"
+F 5 "GRM1555C1H220JA01D" H 1575 2575 60  0001 C CNN "Part Number"
+F 6 "CAP CER 22PF 50V 5% NP0 0402" H 1575 2575 60  0001 C CNN "Description"
 	1    1575 2575
 	-1   0    0    1
@@
 F 2 "gsg-modules:0402" H 2913 2725 50  0001 C CNN
 F 3 "" H 2875 2875 50  0000 C CNN
+F 4 "Murata" H 2875 2875 60  0001 C CNN "Manufacturer"
+F 5 "GRM1555C1H330JA01D" H 2875 2875 60  0001 C CNN "Part Number"
+F 6 "CAP CER 33PF 50V 5% NP0 0402" H 2875 2875 60  0001 C CNN "Description"
 	1    2875 2875
 	0    1    1    0
@@
 F 2 "noob:GSG-B0310J50100AHF" H 5325 6125 60  0001 C CNN
 F 3 "" H 5325 6125 60  0000 C CNN
+F 4 "Anaren" H 5325 6125 60  0001 C CNN "Manufacturer"
+F 5 "B0310J50100AHF" H 5325 6125 60  0001 C CNN "Part Number"
+F 6 "Ultra Low Profile 0805 Balun 50 to 100 ohm Balanced" H 5325 6125 60  0001 C CNN "Description"
 	1    5325 6125
 	1    0    0    -1
@@
 F 2 "gsg-modules:SKY13350-385LF" H 6400 6475 60  0001 C CNN
 F 3 "" H 6400 6475 60  0000 C CNN
+F 4 "Skyworks" H 6400 6475 60  0001 C CNN "Manufacturer"
+F 5 "SKY13350-385LF" H 6400 6475 60  0001 C CNN "Part Number"
+F 6 "0.01-6.0 GHz GaAs SPDT Switch" H 6400 6475 60  0001 C CNN "Description"
 	1    6400 6475
 	0    -1   -1   0
@@
 F 2 "gsg-modules:SKY13350-385LF" H 1650 6700 60  0001 C CNN
 F 3 "" H 1650 6700 60  0000 C CNN
+F 4 "Skyworks" H 1650 6700 60  0001 C CNN "Manufacturer"
+F 5 "SKY13350-385LF" H 1650 6700 60  0001 C CNN "Part Number"
+F 6 "0.01-6.0 GHz GaAs SPDT Switch" H 1650 6700 60  0001 C CNN "Description"
 	1    1650 6700
 	0    -1   -1   0
@@
 F 2 "gsg-modules:0402" H 2363 6375 50  0001 C CNN
 F 3 "" H 2325 6525 50  0000 C CNN
+F 4 "Murata" H 2325 6525 60  0001 C CNN "Manufacturer"
+F 5 "GRM1555C1H220JA01D" H 2325 6525 60  0001 C CNN "Part Number"
+F 6 "CAP CER 22PF 50V 5% NP0 0402" H 2325 6525 60  0001 C CNN "Description"
 	1    2325 6525
 	-1   0    0    -1
@@
 F 2 "gsg-modules:0402" H 1988 5875 50  0001 C CNN
 F 3 "" H 1950 6025 50  0000 C CNN
+F 4 "Murata" H 1950 6025 60  0001 C CNN "Manufacturer"
+F 5 "GRM1555C1H330JA01D" H 1950 6025 60  0001 C CNN "Part Number"
+F 6 "CAP CER 33PF 50V 5% NP0 0402" H 1950 6025 60  0001 C CNN "Description"
 	1    1950 6025
 	0    1    1    0
@@
 F 2 "gsg-modules:0402" H 1213 5875 50  0001 C CNN
 F 3 "" H 1175 6025 50  0000 C CNN
+F 4 "Murata" H 1175 6025 60  0001 C CNN "Manufacturer"
+F 5 "GRM1555C1H220JA01D" H 1175 6025 60  0001 C CNN "Part Number"
+F 6 "CAP CER 22PF 50V 5% NP0 0402" H 1175 6025 60  0001 C CNN "Description"
 	1    1175 6025
 	0    1    1    0
@@
 F 2 "gsg-modules:0402" H 1113 7100 50  0001 C CNN
 F 3 "" H 1075 7250 50  0000 C CNN
+F 4 "Murata" H 1075 7250 60  0001 C CNN "Manufacturer"
+F 5 "GRM1555C1H330JA01D" H 1075 7250 60  0001 C CNN "Part Number"
+F 6 "CAP CER 33PF 50V 5% NP0 0402" H 1075 7250 60  0001 C CNN "Description"
 	1    1075 7250
 	0    -1   -1   0
@@
 F 2 "noob:GSG-HP-DEA" H 11025 4800 60  0001 C CNN
 F 3 "" H 11025 4800 60  0000 C CNN
+F 4 "TDK" H 11025 4800 60  0001 C CNN "Manufacturer"
+F 5 "DEA162400HT-8004B1" H 11025 4800 60  0001 C CNN "Part Number"
+F 6 "FILTER HIGHPASS WLAN&BLUETOOTH" H 11025 4800 60  0001 C CNN "Description"
 	1    11025 4800
 	1    0    0    -1
@@
 F 2 "noob:GSG-LP0603" H 11025 3650 60  0001 C CNN
 F 3 "" H 11025 3650 60  0000 C CNN
+F 4 "AVX" H 11025 3650 60  0001 C CNN "Manufacturer"
+F 5 "LP0603A1880ANTR" H 11025 3650 60  0001 C CNN "Part Number"
+F 6 "FILTER LOW PASS 1880MHZ 0603 SMD" H 11025 3650 60  0001 C CNN "Description"
 	1    11025 3650
 	-1   0    0    1
@@
 F 2 "gsg-modules:SKY13350-385LF" H 12550 4475 60  0001 C CNN
 F 3 "" H 12550 4475 60  0000 C CNN
+F 4 "Skyworks" H 12550 4475 60  0001 C CNN "Manufacturer"
+F 5 "SKY13350-385LF" H 12550 4475 60  0001 C CNN "Part Number"
+F 6 "0.01-6.0 GHz GaAs SPDT Switch" H 12550 4475 60  0001 C CNN "Description"
 	1    12550 4475
 	0    1    1    0
@@
 F 2 "gsg-modules:SKY13317-373LF" H 14525 3525 60  0001 C CNN
 F 3 "" H 14525 3525 60  0000 C CNN
+F 4 "Skyworks" H 14525 3525 60  0001 C CNN "Manufacturer"
+F 5 "SKY13317-373LF" H 14525 3525 60  0001 C CNN "Part Number"
+F 6 "20 MHz-6.0 GHz pHEMT GaAs SP3T Switch" H 14525 3525 60  0001 C CNN "Description"
 	1    14525 3525
 	-1   0    0    1
@@
 F 2 "gsg-modules:SKY13317-373LF" H 8250 7250 60  0001 C CNN
 F 3 "" H 8250 7250 60  0000 C CNN
+F 4 "Skyworks" H 8250 7250 60  0001 C CNN "Manufacturer"
+F 5 "SKY13317-373LF" H 8250 7250 60  0001 C CNN "Part Number"
+F 6 "20 MHz-6.0 GHz pHEMT GaAs SP3T Switch" H 8250 7250 60  0001 C CNN "Description"
 	1    8250 7250
 	1    0    0    -1
@@
 F 2 "gsg-modules:SOT23GDS" H 9100 8525 60  0001 C CNN
 F 3 "" H 9100 8525 60  0000 C CNN
+F 4 "Fairchild" H 9100 8525 60  0001 C CNN "Manufacturer"
+F 5 "BSS84" H 9100 8525 60  0001 C CNN "Part Number"
+F 6 "MOSFET P-CH 50V 130MA SOT-23" H 9100 8525 60  0001 C CNN "Description"
 	1    9100 8525
 	-1   0    0    1
@@
 F 2 "gsg-modules:0402" H 14150 8375 60  0001 C CNN
 F 3 "" H 14150 8375 60  0000 C CNN
+F 4 "Murata" H 14150 8375 60  0001 C CNN "Manufacturer"
+F 5 "LXES15AAA1-100" H 14150 8375 60  0001 C CNN "Part Number"
+F 6 "TVS DIODE ESD .05PF 15KV 0402" H 14150 8375 60  0001 C CNN "Description"
 	1    14150 8375
 	0    1    1    0
@@
 F 2 "gsg-modules:0402" H 3113 8325 50  0001 C CNN
 F 3 "" H 3075 8475 50  0000 C CNN
+F 4 "Murata" H 3075 8475 60  0001 C CNN "Manufacturer"
+F 5 "GRM1555C1H330JA01D" H 3075 8475 60  0001 C CNN "Part Number"
+F 6 "CAP CER 33PF 50V 5% NP0 0402" H 3075 8475 60  0001 C CNN "Description"
 	1    3075 8475
 	1    0    0    1
@@
 F 2 "gsg-modules:0402" H 3438 8325 50  0001 C CNN
 F 3 "" H 3400 8475 50  0000 C CNN
+F 4 "Murata" H 3400 8475 60  0001 C CNN "Manufacturer"
+F 5 "GRM155R71C103KA01D" H 3400 8475 60  0001 C CNN "Part Number"
+F 6 "CAP CER 10000PF 16V 10% X7R 0402" H 3400 8475 60  0001 C CNN "Description"
 	1    3400 8475
 	1    0    0    1
