File: mcu.sch (KiCad schematic (older format))
At the start: 93 parts, among them J1 GSG-USB-MICRO-B-SHIELDED, P61 CONN_1, P62 CONN_1, P63 CONN_1, P64 CONN_1, P65 CONN_1, P66 CONN_1, P67 CONN_1, P68 CONN_1, P69 I2S, P70 CONN_1, P71 GPIO, P72 LPC_JTAG, P73 CONN_1, P74 CONN_1, P75 CONN_11X2, P76 CONN_1, P77 CONN_1, P78 CONN_1, P79 LPC_ISP, SW1 DFU, SW2 RESET, U19 W25Q80BV, U20 LXES1TBCC2-004, U21 LPC43XXFBD144, X2 RTC_XTAL, X3 MCU_XTAL

Commit message: Add files via upload
Noob-sdr v1.0
Connections:
- net FPGA_TCK: now also P71.21 (P21); no longer P71.17 (P17)
- net !VAA_ENABLE: now reaches U21.37 (P5_0)
- net MGTAVTT: no longer names the net of P71.20 (P20)
